File: GW4302.kicad_pcb (KiCad board)
At the start: 4 copper layers, 57.9 x 60.3 mm, 82 parts, among them J1 C64, J2 microUSB, J3 JTAG, U1 74AHC245PW, U10 74AHC125PW, U13 CH340G, U2 74AHC245PW, U3 LD1117S33, U4 74AHC245PW, U5 74AHC245PW, U6 74AHC125PW, U8 LCMXO2-640-TG100, U9 W9825G6KH-6, Y1 12M

Commit message: Done?
Parts:
- removed R15, R23, R4: 1k, stdpads:R_0603
- added C36: 2u2, stdpads:C_0603, F.Cu at (137.0, 43.4)
- added G***: LOGO, LOGO, B.Cu at (148.3, 56.0)
- added G***: LOGO, LOGO, B.Cu at (148.3, 61.3)
- J2: footprint stdpads:USB_Micro-B_ShouHan_MicroXNJ -> stdpads:USB_Micro-B_Amphenol_10118192-0001
- moved D1 10.6 mm to (156.2, 40.0)
- moved R22 5.84 mm to (153.6, 40.0)
- moved R16 3.71 mm to (140.6, 44.9), turned to 0 degrees
- moved H3 3.59 mm to (159.1, 41.3)
- moved C34 2.31 mm to (140.6, 43.4), turned to 0 degrees
- moved J2 1.34 mm to (134.9, 38.6), turned to 180 degrees
- moved R2 0.78 mm to (137.0, 44.9)
Connections:
- U13 pad 10: Net-(U13-Pad10) -> +3V3
- U13 pad 11: Net-(U13-Pad10) -> +3V3
- U13 pad 12: Net-(U13-Pad10) -> +3V3
- U13 pad 15: Net-(R15-Pad1) -> GND
- U13 pad 3: Net-(R4-Pad2) -> +3V3
Routing:
- net Net-(U13-Pad10): track 19.4 -> 0.00 mm
- net /TDO: track 68.0 -> 60.5 mm
- net /~{LED}: track 94.0 -> 100.5 mm
- net Net-(U10-4~{OE}): track 29.7 -> 23.4 mm
- net Net-(R15-Pad1): track 6.14 -> 0.00 mm, vias 2 -> 0
- net GND: track 164.3 -> 170.4 mm
- net +3V3: track 387.9 -> 392.6 mm, vias 117 -> 121
- net Net-(R4-Pad2): track 2.70 -> 0.00 mm, vias 1 -> 0
- net /TDI: track 54.5 -> 53.2 mm
- net /USB5V: track 2.77 -> 3.70 mm
- net Net-(J2-D+): track 35.8 -> 36.5 mm
- net Net-(J2-D-): track 36.1 -> 36.6 mm
Other:
- rule pad_to_mask_clearance: 0.075 -> 0.0762
- board text added: "A10"
- board text removed: "16 MB REU"
- board text removed: "4302A"
- board text removed: "GW"
- board text removed: "Garrett’s Workshop"
- board text removed: "for C64"

Commit message: New version
Parts:
- removed the C3 at (106.2, 62.1)
- removed the C30 at (110.2, 47.0)
- removed the C31 at (116.7, 40.8)
- removed the C32 at (108.8, 54.9)
- removed the C33 at (106.0, 51.4)
- removed the C34 at (140.6, 43.4)
- removed the C4 at (109.7, 62.1)
- removed the C5 at (106.2, 59.9)
- removed the C7 at (148.0, 45.6)
- removed the G*** at (148.3, 61.3)
- removed the U8 at (122.0, 65.3)
- added C10: 10u, stdpads:C_0805, F.Cu at (114.3, 44.0)
- added C11: 10u, stdpads:C_0805, F.Cu at (111.5, 40.5)
- added C12: 10u, stdpads:C_0805, F.Cu at (116.0, 50.9)
- added C23: 2u2, stdpads:C_0603, F.Cu at (107.5, 51.2)
- added C24: 2u2, stdpads:C_0603, F.Cu at (120.7, 77.1)
- added C25: 2u2, stdpads:C_0603, F.Cu at (127.2, 71.7)
- added C26: 2u2, stdpads:C_0603, F.Cu at (137.7, 71.7)
- added C27: 2u2, stdpads:C_0603, F.Cu at (148.1, 71.7)
- added C28: 2u2, stdpads:C_0603, F.Cu at (158.7, 69.7)
- added C37: 22p, stdpads:C_0603, F.Cu at (123.4, 41.0)
- added C38: 22p, stdpads:C_0603, F.Cu at (129.6, 40.8)
- added C39: 22p, stdpads:C_0603, F.Cu at (120.0, 40.2)
- added C40: 2u2, stdpads:C_0603, F.Cu at (124.2, 49.5)
- added J4: BTN, stdpads:PinHeader_1x03_P2.00mm_Vertical, F.Cu at (117.0, 45.1)
- added R15: 3k3, stdpads:R_0603, F.Cu at (106.7, 75.8)
- added R23: DNP, stdpads:R_0603, F.Cu at (120.0, 41.6)
- added R24: 47, stdpads:R_0603, F.Cu at (120.0, 46.0)
- added R25: DNP, stdpads:R_0603, F.Cu at (120.0, 48.9)
- added R26: 47, stdpads:R_0603, F.Cu at (120.0, 47.4)
- added R27: 3k3, stdpads:R_0603, F.Cu at (119.0, 51.8)
- added R28: 1k, stdpads:R_0603, F.Cu at (123.2, 45.4)
- added R4: 10k, stdpads:R_0603, F.Cu at (139.9, 49.2)
- added U1: LCMXO2-640-TG100, stdpads:TQFP-100_14x14mm_P0.5mm, F.Cu at (117.0, 62.8)
- added U11: 74LVC245APW, stdpads:TSSOP-20_4.4x6.5mm_P0.65mm, F.Cu at (142.0, 73.8)
- added U12: 74LVC245APW, stdpads:TSSOP-20_4.4x6.5mm_P0.65mm, F.Cu at (152.4, 73.8)
- added U14: 74LVC1G17GW, stdpads:SOT-353, F.Cu at (107.1, 54.0)
- added U15: XC6206P332MR, stdpads:SOT-23, F.Cu at (111.5, 43.8)
- added U16: LM66200DRL, stdpads:SOT-583, F.Cu at (111.5, 47.5)
- added U5: 74AHCT125PW, stdpads:TSSOP-14_4.4x5mm_P0.65mm, F.Cu at (117.3, 82.0)
- C1, C2, C6: value 10u -> 2u2; footprint stdpads:C_0805 -> stdpads:C_0603
- C9: value 2u2 -> 10u; footprint stdpads:C_0603 -> stdpads:C_0805
- H1, H2, H3, H4, H5: value (none) -> ~
- J3: footprint Connector:Tag-Connect_TC2050-IDC-FP_2x05_P1.27mm_Vertical -> stdpads:Tag-Connect_TC2050-IDC-FP_2x05_P1.27mm_Vertical
- R16: value 10k -> 3k3
- R17, R18, R19, R20: value 1k -> 3k3
- R2, R21: value 1k -> 47
- R3: value 1k -> 10k
- R8: value 10k -> DNP
- U10: value 74AHC125PW -> 74LVC245APW; footprint stdpads:TSSOP-14_4.4x5mm_P0.65mm -> stdpads:TSSOP-20_4.4x6.5mm_P0.65mm
- U3: value LD1117S33 -> W25Q128JVSIQ; footprint stdpads:SOT-223 -> stdpads:SOIC-8_5.3mm
- U4: renamed from U6; value 74AHC125PW -> 74AHCT125PW
- U6: renamed from U5; value 74AHC245PW -> 74LVC245APW
- U7: renamed from U2; value 74AHC245PW -> 74AHCT573PW
- U8: renamed from U1; value 74AHC245PW -> 74AHCT573PW
- U9: renamed from U4; value 74AHC245PW -> 74AHCT573PW
- moved C9 37.8 mm to (108.3, 44.0), turned to 90 degrees
- moved R16 36.9 mm to (136.8, 81.7)
- moved R11 34.2 mm to (109.6, 75.8), turned to -90 degrees
- moved R12 34.0 mm to (111.0, 75.8), turned to -90 degrees
- moved U3 33.7 mm to (138.9, 55.7), turned to 0 degrees
- moved C8 32.6 mm to (114.0, 47.7)
- moved U10 30.9 mm to (131.6, 73.8)
- moved R21 30.4 mm to (127.0, 55.4)
- moved R22 29.1 mm to (127.2, 52.2), turned to 180 degrees
- moved C17 28.6 mm to (110.4, 53.0), turned to 180 degrees
- moved C18 26.7 mm to (107.0, 59.0), turned to -90 degrees
- moved C19 25.7 mm to (107.0, 67.5), turned to 90 degrees
- moved R3 25.6 mm to (138.7, 61.2), turned to 180 degrees
- moved C16 25.0 mm to (113.5, 53.0), turned to 0 degrees
- moved D1 23.4 mm to (132.8, 40.1), turned to 180 degrees
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- renumbered C24 to C29, C10 to C3, C25 to C30, C26 to C31, C27 to C32, C28 to C33, C29 to C34, C23 to C36, C11 to C4, C12 to C5, C36 to C7, U9 to U2
Connections:
- C1 pad 1: +5V -> C5V
- C2 pad 1: +5V -> C5V
- C3 pad 1: +3V3 -> C5V
- C4 pad 1: +3V3 -> C5V
- C5 pad 1: +3V3 -> C5V
- C6 pad 1: +3V3 -> C5V
- C7 pad 1: /USB5V -> U5V
- C8 pad 1: +3V3 -> U5V
- C9 pad 1: +3V3 -> +5V
- D1 pad 1: /~{LED} -> Net-(D1-K)
- D1 pad 2: Net-(D1-A) -> +3V3
- J1 pad 2: +5V -> C5V
- J1 pad 3: +5V -> C5V
- J1 pad 42: /~{RESET} -> /~{RES}
- J2 pad 1: /USB5V -> U5V
- J3 pad 1: /TCK -> /CTCKr
- J3 pad 3: /TMS -> /CTMS
- J3 pad 5: /TDI -> /CTDI
- R1 pad 2: Net-(U5-B5) -> Net-(U6-B4)
- R10 pad 1: /TCKr -> /CTCK
- R10 pad 2: /TCK -> /CTCKr
- R12 pad 1: /~{INIT} -> /O~{EXROM}
- R13 pad 2: /TCKr -> /CTCK
- R14 pad 1: /TMS -> /CTMS
- R16 pad 1: Net-(U10-4~{OE}) -> /O~{NMI}
- R16 pad 2: GND -> +3V3
- R17 pad 1: /A~{OE} -> /Aout~{OE}
- R18 pad 1: /IRQ~{OE} -> /O~{IRQ}
- R19 pad 1: /D~{OE} -> /Dout~{OE}
- R2 pad 1: Net-(U10-4~{OE}) -> /TCK
- R2 pad 2: /USB5V -> /UTXD
- R20 pad 1: /DMA~{OE} -> /O~{DMA}
- R21 pad 1: /RW~{OE} -> /FSCKr
- R21 pad 2: +3V3 -> /FSCK
- R22 pad 1: +3V3 -> Net-(D1-K)
- R22 pad 2: Net-(D1-A) -> /~{LED}
- R3 pad 1: /JTAG~{OE} -> /F~{WP}
- R3 pad 2: GND -> +3V3
- R5 pad 1: +5V -> C5V
- R8 pad 1: GND -> /TMS
- R8 pad 2: /RA4 -> /CTMS
- R9 pad 1: /~{PROG} -> /~{LED}
- U10 pad 1: /JTAG~{OE} -> GND
- U10 pad 10: /JTAG~{OE} -> GND
- U10 pad 11: /JTAG~{OE} -> /A8
- U10 pad 12: +3V3 -> /A9
- U10 pad 13: Net-(U10-4~{OE}) -> /A10
- U10 pad 14: +3V3 -> /A11
- U10 pad 2: /UTDI -> /BA15
- U10 pad 3: /TDI -> /BA14
- U10 pad 4: /JTAG~{OE} -> /BA13
- U10 pad 5: /UTMS -> /BA12
- U10 pad 6: /TMS -> /BA11
- U10 pad 7: GND -> /BA10
- U10 pad 8: /TCKr -> /BA9
- U10 pad 9: /UTCK -> /BA8
- U13 pad 2: /UTCK -> /UTXD
- U13 pad 3: +3V3 -> /FTXD
- U2 pad 10: /RD5 -> /BD5
- U2 pad 11: /RD6 -> /BD6
- U2 pad 13: /RD7 -> /BD7
- U2 pad 19: /R~{CS} -> GND
- U2 pad 2: /RD0 -> /BD0
- U2 pad 4: /RD1 -> /BD1
- U2 pad 40: (no net) -> unconnected-(U2-NC-Pad40)
- U2 pad 42: /RD7 -> /BD7
- U2 pad 44: /RD6 -> /BD6
- U2 pad 45: /RD5 -> /BD5
- U2 pad 47: /RD4 -> /BD4
- U2 pad 48: /RD3 -> /BD3
- U2 pad 5: /RD2 -> /BD2
- U2 pad 50: /RD2 -> /BD2
- U2 pad 51: /RD1 -> /BD1
- U2 pad 53: /RD0 -> /BD0
- U2 pad 7: /RD3 -> /BD3
- U2 pad 8: /RD4 -> /BD4
- U3 pad 1: GND -> /F~{CS}
- U3 pad 2: +3V3 -> /FMISO
- U3 pad 3: +5V -> /F~{WP}
- U4 pad 1: GND -> /O~{RES}
- U4 pad 10: /DMA~{OE} -> /O~{NMI}
- U4 pad 11: /~{IRQ} -> GND
- U4 pad 13: /IRQ~{OE} -> GND
- U4 pad 14: +3V3 -> C5V
- U4 pad 3: unconnected-(U6-1Y-Pad3) -> /~{RES}
- U4 pad 4: /RW~{OE} -> /O~{IRQ}
- U4 pad 5: /DMAR~{W} -> GND
- U4 pad 6: /R~{W} -> /~{IRQ}
- U4 pad 8: /~{DMA} -> /~{NMI}
- U6 pad 12: /B~{IO2} -> /B~{ROML}
- U6 pad 13: Net-(U5-B5) -> /B~{IO}2
- U6 pad 14: /B~{RESET} -> Net-(U6-B4)
- U6 pad 15: /B~{IO1} -> /B~{IO}1
- U6 pad 16: /BR~{W} -> /B~{ROMH}
- U6 pad 17: GND -> /BR~{W}
- U6 pad 3: GND -> /R~{W}
- U6 pad 4: /R~{W} -> /~{ROMH}
- U6 pad 6: /~{RESET} -> /PHI2
- U6 pad 7: /PHI2 -> /~{IO2}
- U6 pad 8: /~{IO2} -> /~{ROML}
- U7 pad 1: /ADIR -> /Aout~{OE}
- U7 pad 11: /BA8 -> +3V3
- U7 pad 12: /BA9 -> /A15
- U7 pad 13: /BA10 -> /A14
- U7 pad 14: /BA11 -> /A13
- U7 pad 15: /BA12 -> /A12
- U7 pad 16: /BA13 -> /A11
- U7 pad 17: /BA14 -> /A10
- U7 pad 18: /BA15 -> /A9
- U7 pad 19: /A~{OE} -> /A8
- U7 pad 2: /A15 -> /BA8
- U7 pad 20: +3V3 -> C5V
- U7 pad 3: /A14 -> /BA9
- U7 pad 4: /A13 -> /BA10
- U7 pad 5: /A12 -> /BA11
- U7 pad 6: /A11 -> /BA12
- U7 pad 7: /A10 -> /BA13
- U7 pad 8: /A9 -> /BA14
- U7 pad 9: /A8 -> /BA15
- U8 pad 1: /ADIR -> /Aout~{OE}
- U8 pad 11: /BA0 -> +3V3
- U8 pad 12: /BA1 -> /A7
- U8 pad 13: /BA2 -> /A6
- U8 pad 14: /BA3 -> /A5
- U8 pad 15: /BA4 -> /A4
- U8 pad 16: /BA5 -> /A3
- U8 pad 17: /BA6 -> /A2
- U8 pad 18: /BA7 -> /A1
- U8 pad 19: /A~{OE} -> /A0
- U8 pad 2: /A7 -> /BA0
- U8 pad 20: +3V3 -> C5V
- U8 pad 3: /A6 -> /BA1
- U8 pad 4: /A5 -> /BA2
- U8 pad 5: /A4 -> /BA3
- U8 pad 6: /A3 -> /BA4
- U8 pad 7: /A2 -> /BA5
- U8 pad 8: /A1 -> /BA6
- U8 pad 9: /A0 -> /BA7
- U9 pad 1: /DDIR -> /Dout~{OE}
- U9 pad 11: /BD0 -> /DLE
- U9 pad 12: /BD1 -> /D7
- U9 pad 13: /BD2 -> /D6
- U9 pad 14: /BD3 -> /D5
- U9 pad 15: /BD4 -> /D4
- U9 pad 16: /BD5 -> /D3
- U9 pad 17: /BD6 -> /D2
- U9 pad 18: /BD7 -> /D1
- U9 pad 19: /D~{OE} -> /D0
- U9 pad 2: /D7 -> /BD0
- U9 pad 20: +3V3 -> C5V
- U9 pad 3: /D6 -> /BD1
- U9 pad 4: /D5 -> /BD2
- U9 pad 5: /D4 -> /BD3
- U9 pad 6: /D3 -> /BD4
- U9 pad 7: /D2 -> /BD5
- U9 pad 8: /D1 -> /BD6
- U9 pad 9: /D0 -> /BD7
Routing:
- net +3V3: track 392.6 -> 159.4 mm, vias 121 -> 103
- net C5V: track 0.00 -> 202.6 mm, vias 0 -> 21
- net /~{LED}: track 100.5 -> 25.9 mm
- net /D~{OE}: track 58.5 -> 0.00 mm, vias 2 -> 0
- net U5V: track 0.00 -> 58.0 mm, vias 0 -> 5
- net +5V: track 57.5 -> 0.00 mm, vias 2 -> 0
- net /DDIR: track 56.0 -> 0.00 mm, vias 2 -> 0
- net GND: track 170.4 -> 218.9 mm, vias 272 -> 290
- net /TCKr: track 48.1 -> 0.00 mm, vias 3 -> 0
- net /CTMS: track 0.00 -> 47.5 mm, vias 0 -> 5
- net /CTDI: track 0.00 -> 47.2 mm, vias 0 -> 4
- net /Aout~{OE}: track 0.00 -> 46.5 mm, vias 0 -> 2
- net /Dout~{OE}: track 0.00 -> 45.7 mm, vias 0 -> 2
- net /~{RES}: track 0.00 -> 43.3 mm, vias 0 -> 3
- net /R~{CS}: track 43.3 -> 0.00 mm
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- added copper zone on F.Cu, net +5V
- added copper zone on F.Cu, net C5V
Other:
- board size 57.9 x 60.3 mm -> 57.9 x 59.4 mm
